Commit message: valid

File: description/urdf/pioneer3at.urdf.xacro (robot description, xacro)
@@ -1,399 +1,13 @@
 <?xml version="1.0"?>
-<!-- Revolute-Revolute Manipulator -->
-<!--this file include visual and geometry messages about p3at-->
-<robot name="pioneer3at" xmlns:xacro="http://www.ros.org/wiki/xacro">
-	<!-- Constants for robot dimensions -->
-	<xacro:property name="PI" value="3.1415926535897931"/>
-	<xacro:property name="width" value="0.1" /> <!-- Square dimensions (widthxwidth) of beams -->
-	<xacro:property name="camera_link" value="0.05" /> <!-- Size of square 'camera' box -->
-	<xacro:property name="axel_offset" value="0.05" /> <!-- Space btw top of beam and the each joint -->
-	<!-- Import all Gazebo-customization elements, including Gazebo colors -->
-	<!--the file below include messages about Gazebo plugins for p3at-->
-	<xacro:include filename="$(find zs_description)/urdf/include/p3at_add/pioneer3at.xacro" />
-	<!-- Import Rviz colors -->
-	<xacro:include filename="$(find zs_description)/urdf/include/p3at_add/materials.xacro" />
-	<!-- Import xacro:macro for wheels -->
-	<xacro:include filename="$(find zs_description)/urdf/include/p3at_add/pioneer3at_wheels.xacro" />
-	<!-- Import xacro:macro for pilars -->
-	<xacro:include filename="$(find zs_description)/urdf/include/p3at_add/pioneer3at_pilars.xacro" />
-	<!-- Chassis -->
-	<link name="base_link">
-		<inertial>
-			<mass value="10.0"/>
-			<origin xyz="0 0 0.177"/>
-			<inertia ixx="0.3338" ixy="0.0" ixz="0.0"
-				 iyy="0.4783" iyz="0.0"
-				 izz="0.3338"/>
-		</inertial>
-		<visual name="base_visual">
-			<origin xyz="0 0 0.177" rpy="0 0 0"/>
-			<geometry name="pioneer_geom">
-				<mesh filename="package://zs_description/meshes/p3at/chassis.stl"/>
-			</geometry>
-			<material name="ChassisRed">
-				<color rgba="0.851 0.0 0.0 1.0"/>
-			</material>
-		</visual>
-		<collision>
-			<origin xyz="0 0 0.177" rpy="0 0 0"/>
-				<geometry>
-					<mesh filename="package://zs_description/meshes/p3at/chassis.stl"/>
-				</geometry>
-		</collision>
-	</link>
-	<!-- Top -->
-	<link name="top_plate">
-		<inertial>
-			<mass value="0.1"/>
-			<origin xyz="-0.025 0 -0.223"/>
-			<inertia ixx="1.0" ixy="0.0" ixz="0.0"
-				 iyy="1.0" iyz="0.0"
- 				izz="1.0"/>
-		</inertial>
-		<visual name="top_visual">
-			<origin xyz="0 0 0" rpy="0 0 0"/>
-			<geometry name="pioneer_geom">
-				<mesh filename="package://zs_description/meshes/p3at/top.stl"/>
-			</geometry>
-			<material name="TopBlack">
-					<color rgba="0.038 0.038 0.038 1.0"/>
-			</material>
-		</visual>
-		<collision>
-			<origin xyz="0 0 0" rpy="0 0 0"/>
-			<geometry>
-				<box size="0 0 0"/>
-			</geometry>
-		</collision>
-	</link>
-	<joint name="base_top_joint" type="fixed">
-		<origin xyz="0.003 0 0.274" rpy="0 0 0"/>
-		<parent link="base_link"/>
-		<child link="top_plate"/>
-	</joint>
-	<!-- Long pilars -->
-	<xacro:longpilar_front suffix="left" reflect="1"/>
-	<xacro:longpilar_front suffix="right" reflect="-1"/>
-	<!-- Side_left -->
-	<link name="side_plate_left">
-		<inertial>
-			<mass value="0.1"/>
-			<origin xyz="0 0 0"/>
-			<inertia ixx="1.0" ixy="0.0" ixz="0.0"
-				 iyy="1.0" iyz="0.0"
- 				izz="1.0"/>
-		</inertial>
-		<visual name="side_visual">
-			<origin xyz="0 0 0" rpy="1.57079 0 0"/>
-			<geometry name="pioneer_geom">
-				<mesh filename="package://zs_description/meshes/lateral/lateral.stl"/>
-			</geometry>
-			<material name="ChassisRed">
-				<color rgba="0.8 0.0 0.0 1.0"/>
-			</material>
-		</visual>
-		<collision>
-			<origin xyz="0 0 0" rpy="1.57079 0 0"/>
-			<geometry>
-				<mesh filename="package://zs_description/meshes/lateral/lateral.stl"/>
-			</geometry>
-		</collision>
-	</link>
-	<joint name="base_sideleft_joint" type="fixed">
-		<origin xyz="-0.02 0.165 0.1" rpy="0 0 0"/>
-		<parent link="top_plate"/>
-		<child link="side_plate_left"/>
-	</joint>
-		<!-- Side_right -->
-	<link name="side_plate_right">
-		<inertial>
-			<mass value="0.1"/>
-			<origin xyz="0 0 0"/>
-			<inertia ixx="1.0" ixy="0.0" ixz="0.0"
-				 iyy="1.0" iyz="0.0"
- 				izz="1.0"/>
-		</inertial>
-		<visual name="side_visual">
-			<origin xyz="0 0 0" rpy="1.57079 0 0"/>
-			<geometry name="pioneer_geom">
-				<mesh filename="package://zs_description/meshes/lateral/lateral.stl"/>
-			</geometry>
-			<material name="ChassisRed">
-				<color rgba="0.8 0.0 0.0 1.0"/>
-			</material>
-		</visual>
-		<collision>
-			<origin xyz="0 0 0" rpy="1.57079 0 0"/>
-			<geometry>
-				<mesh filename="package://zs_description/meshes/lateral/lateral.stl"/>
-			</geometry>
-		</collision>
-	</link>
-	<joint name="base_sideright_joint" type="fixed">
-		<origin xyz="-0.02 -0.162 0.1" rpy="0 0 0"/>
-		<parent link="top_plate"/>
-		<child link="side_plate_right"/>
-	</joint>
-		<!-- Side_back_down_right -->
-	<link name="side_plate_back_down_right">
-		<inertial>
-			<mass value="0.1"/>
-			<origin xyz="0 0 0"/>
-			<inertia ixx="1.0" ixy="0.0" ixz="0.0"
-				 iyy="1.0" iyz="0.0"
- 				izz="1.0"/>
-		</inertial>
-		<visual name="side_visual">
-			<origin xyz="0 0 0" rpy="0 0 0"/>
-			<geometry name="pioneer_geom">
-				<box size="0.15 0.003 0.11"/>
-			</geometry>
-			<material name="ChassisRed">
-				<color rgba="0.8 0.0 0.0 1.0"/>
-			</material>
-		</visual>
-		<collision>
-			<origin xyz="0 0 0" rpy="0 0 0"/>
-			<geometry>
-				<box size="0.15 0.003 0.11"/>
-			</geometry>
-		</collision>
-	</link>
-	<joint name="base_sidebackdownright_joint" type="fixed">
-		<origin xyz="-0.205 -0.095 0.055" rpy="0 0 -1.1"/>
-		<parent link="top_plate"/>
-		<child link="side_plate_back_down_right"/>
-	</joint>
-		<!-- Side_back_up_right -->
-	<link name="side_plate_back_up_right">
-		<inertial>
-			<mass value="0.1"/>
-			<origin xyz="0 0 0"/>
-			<inertia ixx="1.0" ixy="0.0" ixz="0.0"
-				 iyy="1.0" iyz="0.0"
- 				izz="1.0"/>
-		</inertial>
-		<visual name="side_visual">
-			<origin xyz="0 0 0" rpy="0 0 0"/>
-			<geometry name="pioneer_geom">
-				<box size="0.15 0.003 0.08"/>
-			</geometry>
-			<material name="ChassisRed">
-				<color rgba="0.8 0.0 0.0 1.0"/>
-			</material>
-		</visual>
-		<collision>
-			<origin xyz="0 0 0" rpy="0 0 0"/>
-			<geometry>
-				<box size="0.15 0.003 0.08"/>
-			</geometry>
-		</collision>
-	</link>
-	<joint name="base_sidebackupright_joint" type="fixed">
-		<origin xyz="-0.205 -0.095 0.16" rpy="0 0 -1.1"/>
-		<parent link="top_plate"/>
-		<child link="side_plate_back_up_right"/>
-	</joint>
-		<!-- Side_back_down_left -->
-	<link name="side_plate_back_down_left">
-		<inertial>
-			<mass value="0.1"/>
-			<origin xyz="0 0 0"/>
-			<inertia ixx="1.0" ixy="0.0" ixz="0.0"
-				 iyy="1.0" iyz="0.0"
- 				izz="1.0"/>
-		</inertial>
-		<visual name="side_visual">
-			<origin xyz="0 0 0" rpy="0 0 0"/>
-			<geometry name="pioneer_geom">
-				<box size="0.15 0.003 0.11"/>
-			</geometry>
-			<material name="ChassisRed">
-				<color rgba="0.8 0.0 0.0 1.0"/>
-			</material>
-		</visual>
-		<collision>
-			<origin xyz="0 0 0" rpy="0 0 0"/>
-			<geometry>
-				<box size="0.15 0.003 0.11"/>
-			</geometry>
-		</collision>
-	</link>
-	<joint name="base_sidebackdownleft_joint" type="fixed">
-		<origin xyz="-0.205 0.095 0.055" rpy="0 0 1.1"/>
-		<parent link="top_plate"/>
-		<child link="side_plate_back_down_left"/>
-	</joint>
-		<!-- Side_back_up_left -->
-	<link name="side_plate_back_up_left">
-		<inertial>
-			<mass value="0.1"/>
-			<origin xyz="0 0 0"/>
-			<inertia ixx="1.0" ixy="0.0" ixz="0.0"
-				 iyy="1.0" iyz="0.0"
- 				izz="1.0"/>
-		</inertial>
-		<visual name="side_visual">
-			<origin xyz="0 0 0" rpy="0 0 0"/>
-			<geometry name="pioneer_geom">
-				<box size="0.15 0.003 0.08"/>
-			</geometry>
-			<material name="ChassisRed">
-				<color rgba="0.8 0.0 0.0 1.0"/>
-			</material>
-		</visual>
-		<collision>
-			<origin xyz="0 0 0" rpy="0 0 0"/>
-			<geometry>
-				<box size="0.15 0.003 0.08"/>
-			</geometry>
-		</collision>
-	</link>
-	<joint name="base_sidebackupleft_joint" type="fixed">
-		<origin xyz="-0.205 0.095 0.16" rpy="0 0 1.1"/>
-		<parent link="top_plate"/>
-		<child link="side_plate_back_up_left"/>
-	</joint>
-		<!-- Side_back_up -->
-	<link name="side_plate_back_up">
-		<inertial>
-			<mass value="0.1"/>
-			<origin xyz="0 0 0"/>
-			<inertia ixx="1.0" ixy="0.0" ixz="0.0"
-				 iyy="1.0" iyz="0.0"
- 				izz="1.0"/>
-		</inertial>
-		<visual name="side_visual">
-			<origin xyz="0 0 0" rpy="0 0 0"/>
-			<geometry name="pioneer_geom">
-				<box size="0.058 0.003 0.05"/>
-			</geometry>
-			<material name="ChassisRed">
-				<color rgba="0.8 0.0 0.0 1.0"/>
-			</material>
-		</visual>
-		<collision>
-			<origin xyz="0 0 0" rpy="0 0 0"/>
-			<geometry>
-				<box size="0.058 0.003 0.05"/>
-			</geometry>
-		</collision>
-	</link>
-	<joint name="base_sidebackup_joint" type="fixed">
-		<origin xyz="-0.24 0. 0.175" rpy="0 0 1.57079"/>
-		<parent link="top_plate"/>
-		<child link="side_plate_back_up"/>
-	</joint>
-	<!-- Top top-->
-	<link name="toptop_plate">
-		<inertial>
-			<mass value="0.1"/>
-			<origin xyz="0 0 0"/>
-			<inertia ixx="1.0" ixy="0.0" ixz="0.0"
-				 iyy="1.0" iyz="0.0"
- 				izz="1.0"/>
-		</inertial>
-		<visual name="toptop_visual">
-			<origin xyz="0 0 0" rpy="0 0 0"/>
-			<geometry name="pioneer_geom">
-				<mesh filename="package://zs_description/meshes/lateral/toptop.stl"/>
-			</geometry>
-			<material name="TopBlack">
-					<color rgba="0.038 0.038 0.038 1.0"/>
-			</material>
-		</visual>
-		<collision>
-			<origin xyz="0 0 0" rpy="0 0 0"/>
-			<geometry>
-				<box size="0 0 0"/>
-			</geometry>
-		</collision>
-	</link>
-	<joint name="base_toptop_joint" type="fixed">
-		<origin xyz="0.003 0 0.2" rpy="0 0 0"/>
-		<parent link="top_plate"/>
-		<child link="toptop_plate"/>
-	</joint>
-	<!-- Sick Laser -->
-	<link name="laser">
-		<collision>
-			<origin xyz="0 0 -0.06" rpy="0 0 0"/>
-			<geometry>
-				<box size="0.1 0.1 0.16"/>
-			</geometry>
-		</collision>
-		<visual>
-			<origin xyz="0 0 -0.05" rpy="3.141592 0 0"/>
-			<geometry>
-				<mesh filename="package://zs_description/meshes/sick_lms1xx/sick_lms100.dae"/>
-			</geometry>
-		</visual>
-		<inertial>
-			<mass value="1e-5" />
-			<inertia ixx="1e-6" ixy="0" ixz="0" iyy="1e-6" iyz="0" izz="1e-6" />
-		</inertial>
-	</link>
-	<joint name="laser_joint" type="fixed">
-		<axis xyz="0 1 0" />
-		<origin xyz="-0.195 0 0.39" rpy="0 0 3.141592"/>
-		<parent link="base_link"/>
-		<child link="laser"/>
-	</joint>
-	<!-- Wheels, axes and hubs -->
-	<xacro:p3at_front suffix="left" reflect="1"/>
-	<xacro:p3at_front suffix="right" reflect="-1"/>
-	<!-- Camera -->
-	<link name="camera_link">
-		<collision>
-			<origin xyz="0 0 0" rpy="0 0 0"/>
-			<geometry>
-				<box size="0.06 0.21 0.070"/>
-			</geometry>
-		</collision>
-		<visual>
-			<origin xyz="0 0 -0.01" rpy="0 0 1.570796"/>
-			<geometry>
-				<mesh filename="package://zs_description/meshes/kinect/kinect.dae"/>
-			</geometry>
-		</visual>
-		<inertial>
-			<mass value="0.546" />
-			<origin xyz="0 0 0" rpy="0 0 0"/>
-			<inertia ixx="0.003881243" ixy="0" ixz="0" iyy="0.000498940" iyz="0" izz="0.003879257" />
-		</inertial>
-	</link>
-	<joint name="camera_joint" type="fixed">
-		<axis xyz="0 1 0" />
-		<origin xyz="0 0 0.10" rpy="0 0 0"/>
-		<parent link="top_plate"/>
-		<child link="camera_link"/>
-	</joint>
-<!-- camera config from turtlebot!! -->
-	<joint name="camera_rgb_joint" type="fixed">
-		<origin xyz="-0.087 -0.0125 0.2870" rpy="0 0 0"/>
-		<parent link="camera_link"/>
-		<child link="camera_rgb_frame"/>
-	</joint>
-	<link name="camera_rgb_frame"/>
-	<joint name="camera_rgb_optical_joint" type="fixed">
-		<origin xyz="0 0 0" rpy="-1.570796 0 -1.570796" />
-		<parent link="camera_rgb_frame" />
-		<child link="camera_rgb_optical_frame" />
-	</joint>
-	<link name="camera_rgb_optical_frame"/>
-    <!-- The fixed joints & links below are usually published by static_transformers launched by the OpenNi launch
-         files. However, for Gazebo simulation we need them, so we add them here.
-         (Hence, don't publish them additionally!) -->
-	<joint name="camera_depth_joint" type="fixed">
-		<origin xyz="0 -0.0250 0" rpy="0 0 0" />
-		<parent link="camera_link" />
-		<child link="camera_depth_frame" />
-	</joint>
-	<link name="camera_depth_frame"/>
-	<joint name="camera_depth_optical_joint" type="fixed">
-		<origin xyz="0 0 0" rpy="-1.570796 0 -1.570796" />
-		<parent link="camera_depth_frame" />
-		<child link="camera_depth_optical_frame" />
-	</joint>
-	<link name="camera_depth_optical_frame"/>
+<robot
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